File: ALU_4Bits.kicad_sch (KiCad schematic)
At the start: 10 parts, among them U701 74HC86, U702 74LS08, U703 74LS32, U704 74HC86, U705 74LS08

Commit message: Working
Parts:
- renumbered C701 to C1301, C702 to C1302, C703 to C1303, C704 to C1304, C705 to C1305, U701 to U1301, U702 to U1302, U703 to U1303, U704 to U1304, U705 to U1305

Commit message: More cleanup and preparing signals for control logic
Parts:
- renumbered C1301 to C301, C1302 to C302, C1303 to C303, C1304 to C304, C1305 to C305, U1301 to U301, U1302 to U302, U1304 to U303, U1305 to U304, U1303 to U305

Commit message: Draft Schematic
Parts:
- C301, C302, C303, C304, C305: value C -> 0.1uF; footprint (none) -> Capacitor_THT:C_Rect_L4.0mm_W2.5mm_P2.50mm
- U301: footprint (none) -> Package_DIP:DIP-14_W7.62mm
- U302: value 74LS08 -> 74HC08; footprint (none) -> Package_DIP:DIP-14_W7.62mm
- U303: renamed from U305; value 74LS32 -> 74HC32; footprint (none) -> Package_DIP:DIP-14_W7.62mm
- U304: renamed from U303; footprint (none) -> Package_DIP:DIP-14_W7.62mm
- U305: renamed from U304; value 74LS08 -> 74HC08; footprint (none) -> Package_DIP:DIP-14_W7.62mm
Other:
- moved on the sheet: C301, C302, C303, C304, C305, U301E, U302E, U303E, U304E, U305E
