File: BRISC8.kicad_sch (KiCad schematic)
At the start: 0 parts

Commit message: Working
Other:
- removed sheet ALU
- removed sheet ProgramCounter
- removed sheet Register0
- removed sheet Register1
- removed sheet Register2
- added sheet BRISC8 CPU (BRISC8 CPU.kicad_sch)

Commit message: Fixed(?)
Other:
- sheet BRISC8 CPU ports: added Addr_{[0..7]}, Clock, Data_{[0..7]}, IO/~{Memory}, Read/~{Write}, ~{Reset}; removed none
Changed lines of the file:
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@@
 	(sheet
 		(at 93.98 53.34)
-		(size 39.37 31.75)
+		(size 24.13 12.7)
 		(exclude_from_sim no)
 		(in_bom yes)
@@
 		)
 		(property "Sheetfile" "BRISC8 CPU.kicad_sch"
-			(at 93.98 85.6746 0)
+			(at 93.98 66.6246 0)
 			(effects
 				(font
@@
 			)
 		)
+		(pin "Data_{[0..7]}" bidirectional
+			(at 118.11 55.88 0)
+			(effects
+				(font
+					(size 1.27 1.27)
+				)
+				(justify right)
+			)
+		)
+		(pin "Addr_{[0..7]}" output
+			(at 118.11 58.42 0)
+			(effects
+				(font
+					(size 1.27 1.27)
+				)
+				(justify right)
+			)
+		)
+		(pin "Read{slash}~{Write}" output
+			(at 118.11 60.96 0)
+			(effects
+				(font
+					(size 1.27 1.27)
+				)
+				(justify right)
+			)
+		)
+		(pin "IO{slash}~{Memory}" output
+			(at 118.11 63.5 0)
+			(effects
+				(font
+					(size 1.27 1.27)
+				)
+				(justify right)
+			)
+		)
+		(pin "Clock" input
+			(at 93.98 55.88 180)
+			(effects
+				(font
+					(size 1.27 1.27)
+				)
+				(justify left)
+			)
+		)
+		(pin "~{Reset}" input
+			(at 93.98 58.42 180)
+			(effects
+				(font
+					(size 1.27 1.27)
+				)
+				(justify left)
+			)
+		)

Commit message: Draft Schematic
Parts:
- added C101: 0.33uF, Capacitor_THT:CP_Radial_D5.0mm_P2.50mm, symbol Device:C_Polarized_Small
- added C102: 10uF, Capacitor_THT:CP_Radial_D5.0mm_P2.00mm, symbol Device:C_Polarized_Small
- added C103: 0.1uF, Capacitor_THT:C_Rect_L4.0mm_W2.5mm_P2.50mm, symbol Device:C_Small
- added D101: PWR, LED_THT:LED_D5.0mm, symbol Device:LED
- added J101: DC In, Connector_BarrelJack:BarrelJack_GCT_DCJ200-10-A_Horizontal, symbol Connector:Barrel_Jack
- added J102: 5V In, TerminalBlock_RND:TerminalBlock_RND_205-00001_1x02_P5.00mm_Horizontal, symbol Connector:Screw_Terminal_01x02
- added R101: 150, Resistor_THT:R_Axial_DIN0207_L6.3mm_D2.5mm_P10.16mm_Horizontal, symbol Device:R
- added U101: L7805, Package_TO_SOT_THT:TO-220-3_Horizontal_TabDown, symbol Regulator_Linear:L7805
Connections:
- new net: C101.1, J101.1, U101.1 (IN)
- new net: D101.1 (K), R101.1
- new net +5V: C102.1, C103.1, D101.2 (A), J102.1 (Pin_1), U101.3 (OUT)
- new net GND: C101.2, C102.2, C103.2, J101.2, J102.2 (Pin_2), R101.2, U101.2 (GND)
Other:
- added sheet Clock & Reset (ClockAndReset.kicad_sch)
- added sheet IO Block (IO Block.kicad_sch)
- added sheet Memory (Memory.kicad_sch)
- sheet BRISC8 CPU ports: added Reset; removed none
