File: InstructionDecode.kicad_sch (KiCad schematic)
At the start: 4 parts, among them U1301 27C256, U1501 74HC161, U1502 74AHC04, U1503 27C256

Commit message: Draft Schematic
Parts:
- added C1501, C1502, C1503, C1504: 0.1uF, Capacitor_THT:C_Rect_L4.0mm_W2.5mm_P2.50mm, symbol Device:C
- U1501: renamed from U1502; value 74AHC04 -> 74HC04; footprint (none) -> Package_DIP:DIP-14_W7.62mm
- U1502: renamed from U1501; footprint (none) -> Package_DIP:DIP-16_W7.62mm
- U1503: renamed from U1301; footprint Package_DIP:DIP-28_W15.24mm -> Package_DIP:DIP-28_W15.24mm_Socket
- U1504: renamed from U1503; footprint Package_DIP:DIP-28_W15.24mm -> Package_DIP:DIP-28_W15.24mm_Socket
Connections:
- net +5V: now also C1501.1, C1502.1, C1503.1, C1504.1
- net GND: now also U1501.11, U1501.13, U1501.5, U1501.9, C1501.2, C1502.2, C1503.2, C1504.2; no longer U1503.2 (A12), U1504.2 (A12)
- net ~{ALU OE}: now reaches U1503.18 (D6)
- net ALU_OP_{0}: now reaches U1504.13 (D2)
- net ALU_OP_{1}: now reaches U1504.15 (D3)
- new net InA_Negative: U1503.2 (A12), U1504.2 (A12)
- no-connect marks 1 -> 9
Other:
- company: (none) -> Brian Duffy
- title: (none) -> BRISC8 CPU
- moved on the sheet: U1501E, U1501F
