File: InstructionRegister.kicad_sch (KiCad schematic)
At the start: 2 parts, among them U301 74HCT173, U302 74HCT173

Commit message: More cleanup and preparing signals for control logic
Parts:
- renumbered U301 to U701, U302 to U702
Changed lines of the file:
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@@
 		(dnp no)
 		(fields_autoplaced yes)
-		(property "Reference" "U301"
+		(property "Reference" "U701"
 			(at 78.3433 53.34 0)
 			(effects
@@
 		(instances
 			(project "BRISC8"
-				(path "/e198223b-f7bd-4b26-ae2e-259db8d07fb6/d081cdcb-1181-4657-9580-dc3ba9a85775/f1dd1a16-fcf9-4d86-90e6-84d5d88c2989"
-					(reference "U301")
+				(path "/e198223b-f7bd-4b26-ae2e-259db8d07fb6/d081cdcb-1181-4657-9580-dc3ba9a85775/2816b318-b467-484f-aabf-89cc6e1c558f"
+					(reference "U701")
 					(unit 1)
 				)
@@
 		(dnp no)
 		(fields_autoplaced yes)
-		(property "Reference" "#PWR0301"
+		(property "Reference" "#PWR0702"
 			(at 76.2 57.15 0)
 			(effects
@@
 		(instances
 			(project "BRISC8"
-				(path "/e198223b-f7bd-4b26-ae2e-259db8d07fb6/d081cdcb-1181-4657-9580-dc3ba9a85775/f1dd1a16-fcf9-4d86-90e6-84d5d88c2989"
-					(reference "#PWR0301")
+				(path "/e198223b-f7bd-4b26-ae2e-259db8d07fb6/d081cdcb-1181-4657-9580-dc3ba9a85775/2816b318-b467-484f-aabf-89cc6e1c558f"
+					(reference "#PWR0702")
 					(unit 1)
 				)
@@
 		(on_board yes)
 		(dnp no)
-		(property "Reference" "#PWR0304"
+		(property "Reference" "#PWR0704"
 			(at 107.95 80.01 0)
 			(effects
@@
 		(instances
 			(project "BRISC8"
-				(path "/e198223b-f7bd-4b26-ae2e-259db8d07fb6/d081cdcb-1181-4657-9580-dc3ba9a85775/f1dd1a16-fcf9-4d86-90e6-84d5d88c2989"
-					(reference "#PWR0304")
+				(path "/e198223b-f7bd-4b26-ae2e-259db8d07fb6/d081cdcb-1181-4657-9580-dc3ba9a85775/2816b318-b467-484f-aabf-89cc6e1c558f"
+					(reference "#PWR0704")
 					(unit 1)
 				)
@@
 		(dnp no)
 		(fields_autoplaced yes)
-		(property "Reference" "#PWR0302"
+		(property "Reference" "#PWR0705"
 			(at 125.73 57.15 0)
 			(effects
@@
 		(instances
 			(project "BRISC8"
-				(path "/e198223b-f7bd-4b26-ae2e-259db8d07fb6/d081cdcb-1181-4657-9580-dc3ba9a85775/f1dd1a16-fcf9-4d86-90e6-84d5d88c2989"
-					(reference "#PWR0302")
+				(path "/e198223b-f7bd-4b26-ae2e-259db8d07fb6/d081cdcb-1181-4657-9580-dc3ba9a85775/2816b318-b467-484f-aabf-89cc6e1c558f"
+					(reference "#PWR0705")
 					(unit 1)
 				)
@@
 		(dnp no)
 		(fields_autoplaced yes)
-		(property "Reference" "#PWR0305"
+		(property "Reference" "#PWR0703"
 			(at 76.2 105.41 0)
 			(effects
@@
 		(instances
 			(project "BRISC8"
-				(path "/e198223b-f7bd-4b26-ae2e-259db8d07fb6/d081cdcb-1181-4657-9580-dc3ba9a85775/f1dd1a16-fcf9-4d86-90e6-84d5d88c2989"
-					(reference "#PWR0305")
+				(path "/e198223b-f7bd-4b26-ae2e-259db8d07fb6/d081cdcb-1181-4657-9580-dc3ba9a85775/2816b318-b467-484f-aabf-89cc6e1c558f"
+					(reference "#PWR0703")
 					(unit 1)
 				)
@@
 		(dnp no)
 		(fields_autoplaced yes)
-		(property "Reference" "U302"
+		(property "Reference" "U702"
 			(at 127.8733 53.34 0)
 			(effects
@@
 		(instances
 			(project "BRISC8"
-				(path "/e198223b-f7bd-4b26-ae2e-259db8d07fb6/d081cdcb-1181-4657-9580-dc3ba9a85775/f1dd1a16-fcf9-4d86-90e6-84d5d88c2989"
-					(reference "U302")
+				(path "/e198223b-f7bd-4b26-ae2e-259db8d07fb6/d081cdcb-1181-4657-9580-dc3ba9a85775/2816b318-b467-484f-aabf-89cc6e1c558f"
+					(reference "U702")
 					(unit 1)
 				)
@@
 		(dnp no)
 		(fields_autoplaced yes)
-		(property "Reference" "#PWR0306"
+		(property "Reference" "#PWR0706"
 			(at 125.73 105.41 0)
 			(effects
@@
 		(instances
 			(project "BRISC8"
-				(path "/e198223b-f7bd-4b26-ae2e-259db8d07fb6/d081cdcb-1181-4657-9580-dc3ba9a85775/f1dd1a16-fcf9-4d86-90e6-84d5d88c2989"
-					(reference "#PWR0306")
+				(path "/e198223b-f7bd-4b26-ae2e-259db8d07fb6/d081cdcb-1181-4657-9580-dc3ba9a85775/2816b318-b467-484f-aabf-89cc6e1c558f"
+					(reference "#PWR0706")
 					(unit 1)
 				)
@@
 		(on_board yes)
 		(dnp no)
-		(property "Reference" "#PWR0303"
+		(property "Reference" "#PWR0701"
 			(at 58.42 80.01 0)
 			(effects
@@
 		(instances
 			(project "BRISC8"
-				(path "/e198223b-f7bd-4b26-ae2e-259db8d07fb6/d081cdcb-1181-4657-9580-dc3ba9a85775/f1dd1a16-fcf9-4d86-90e6-84d5d88c2989"
-					(reference "#PWR0303")
-					(unit 1)
-				)
+				(path "/e198223b-f7bd-4b26-ae2e-259db8d07fb6/d081cdcb-1181-4657-9580-dc3ba9a85775/2816b318-b467-484f-aabf-89cc6e1c558f"
+					(reference "#PWR0701")
+					(unit 1)
+				)

Commit message: Draft Schematic
Parts:
- added C701, C702: 0.1uF, Capacitor_THT:C_Rect_L4.0mm_W2.5mm_P2.50mm, symbol Device:C
- U701, U702: value 74HCT173 -> 74HC173; footprint (none) -> Package_DIP:DIP-16_W7.62mm
Connections:
- net +5V: now also C701.1, C702.1
- net GND: now also C701.2, C702.2
- net Imm_{0} renamed Out_{0}
- net Imm_{1} renamed Out_{1}
- net Imm_{2} renamed Out_{4}
- net Imm_{3} renamed Out_{5}
Other:
- company: (none) -> Brian Duffy
- title: (none) -> BRISC8 CPU
