File: ProgramCounter.kicad_sch (KiCad schematic)
At the start: 8 parts, among them U901 74LS161, U902 74LS161, U903 74HC245, U904 74HC245

Commit message: Draft Schematic
Parts:
- C901, C902, C903, C904: value C -> 0.1uF; footprint (none) -> Capacitor_THT:C_Rect_L4.0mm_W2.5mm_P2.50mm
- U901: renamed from U903; footprint (none) -> Package_DIP:DIP-20_W7.62mm
- U902: renamed from U904; footprint (none) -> Package_DIP:DIP-20_W7.62mm
- U903: renamed from U901; value 74LS161 -> 74HC161; footprint (none) -> Package_DIP:DIP-16_W7.62mm
- U904: renamed from U902; value 74LS161 -> 74HC161; footprint (none) -> Package_DIP:DIP-16_W7.62mm
Changed lines of the file:
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@@
 	(title_block
 		(title "BRISC8 CPU")
-		(date "2025-06-05")
+		(date "2025-06-26")
 		(rev "v1.0.0")
 		(company "Brian Duffy")
@@
 		(dnp no)
 		(fields_autoplaced yes)
-		(property "Reference" "#PWR0901"
+		(property "Reference" "#PWR0905"
 			(at 33.02 62.23 0)
 			(effects
@@
 			(project "BRISC8"
 				(path "/e198223b-f7bd-4b26-ae2e-259db8d07fb6/d081cdcb-1181-4657-9580-dc3ba9a85775/ded358fb-ee52-4096-a32a-0cce52708100/0c7a1bf0-e6ae-42c1-a12c-9c71b98ed1be"
-					(reference "#PWR0901")
+					(reference "#PWR0905")
 					(unit 1)
 				)
@@
 		(on_board yes)
 		(dnp no)
-		(property "Reference" "#PWR0911"
+		(property "Reference" "#PWR0907"
 			(at 208.28 68.58 0)
 			(effects
@@
 			(project "BRISC8"
 				(path "/e198223b-f7bd-4b26-ae2e-259db8d07fb6/d081cdcb-1181-4657-9580-dc3ba9a85775/ded358fb-ee52-4096-a32a-0cce52708100/0c7a1bf0-e6ae-42c1-a12c-9c71b98ed1be"
-					(reference "#PWR0911")
+					(reference "#PWR0907")
 					(unit 1)
 				)
@@
 		(dnp no)
 		(fields_autoplaced yes)
-		(property "Reference" "#PWR0910"
+		(property "Reference" "#PWR0908"
 			(at 161.29 81.28 0)
 			(effects
@@
 			(project "BRISC8"
 				(path "/e198223b-f7bd-4b26-ae2e-259db8d07fb6/d081cdcb-1181-4657-9580-dc3ba9a85775/ded358fb-ee52-4096-a32a-0cce52708100/0c7a1bf0-e6ae-42c1-a12c-9c71b98ed1be"
-					(reference "#PWR0910")
+					(reference "#PWR0908")
 					(unit 1)
 				)
@@
 			)
 		)
-		(property "Value" "C"
+		(property "Value" "0.1uF"
 			(at 113.03 184.1499 0)
 			(effects
@@
 			)
 		)
-		(property "Footprint" ""
+		(property "Footprint" "Capacitor_THT:C_Rect_L4.0mm_W2.5mm_P2.50mm"
 			(at 110.1852 186.69 0)
 			(effects
@@
 		(dnp no)
 		(fields_autoplaced yes)
-		(property "Reference" "#PWR0903"
+		(property "Reference" "#PWR0910"
 			(at 60.96 82.55 0)
 			(effects
@@
 			(project "BRISC8"
 				(path "/e198223b-f7bd-4b26-ae2e-259db8d07fb6/d081cdcb-1181-4657-9580-dc3ba9a85775/ded358fb-ee52-4096-a32a-0cce52708100/0c7a1bf0-e6ae-42c1-a12c-9c71b98ed1be"
-					(reference "#PWR0903")
+					(reference "#PWR0910")
 					(unit 1)
 				)
@@
 		(dnp no)
 		(fields_autoplaced yes)
-		(property "Reference" "#PWR0907"
+		(property "Reference" "#PWR0911"
 			(at 110.49 82.55 0)
 			(effects
@@
 			(project "BRISC8"
 				(path "/e198223b-f7bd-4b26-ae2e-259db8d07fb6/d081cdcb-1181-4657-9580-dc3ba9a85775/ded358fb-ee52-4096-a32a-0cce52708100/0c7a1bf0-e6ae-42c1-a12c-9c71b98ed1be"
-					(reference "#PWR0907")
+					(reference "#PWR0911")
 					(unit 1)
 				)
@@
 		(dnp no)
 		(fields_autoplaced yes)
-		(property "Reference" "#PWR0902"
+		(property "Reference" "#PWR0903"
 			(at 60.96 39.37 0)
 			(effects
@@
 			(project "BRISC8"
 				(path "/e198223b-f7bd-4b26-ae2e-259db8d07fb6/d081cdcb-1181-4657-9580-dc3ba9a85775/ded358fb-ee52-4096-a32a-0cce52708100/0c7a1bf0-e6ae-42c1-a12c-9c71b98ed1be"
-					(reference "#PWR0902")
+					(reference "#PWR0903")
 					(unit 1)
 				)
@@
 			)
 		)
-		(property "Value" "C"
+		(property "Value" "0.1uF"
 			(at 125.73 184.1499 0)
 			(effects
@@
 			)
 		)
-		(property "Footprint" ""
+		(property "Footprint" "Capacitor_THT:C_Rect_L4.0mm_W2.5mm_P2.50mm"
 			(at 122.8852 186.69 0)
 			(effects
@@
 		(dnp no)
 		(fields_autoplaced yes)
-		(property "Reference" "#PWR0909"
+		(property "Reference" "#PWR0901"
 			(at 161.29 38.1 0)
 			(effects
@@
 			(project "BRISC8"
 				(path "/e198223b-f7bd-4b26-ae2e-259db8d07fb6/d081cdcb-1181-4657-9580-dc3ba9a85775/ded358fb-ee52-4096-a32a-0cce52708100/0c7a1bf0-e6ae-42c1-a12c-9c71b98ed1be"
-					(reference "#PWR0909")
+					(reference "#PWR0901")
 					(unit 1)
 				)
@@
 		(dnp no)
 		(fields_autoplaced yes)
-		(property "Reference" "U903"
+		(property "Reference" "U901"
 			(at 163.4333 34.29 0)
 			(effects
@@
 			)
 		)
-		(property "Footprint" ""
+		(property "Footprint" "Package_DIP:DIP-20_W7.62mm"
 			(at 161.29 54.61 0)
 			(effects
@@
 			(project "BRISC8"
 				(path "/e198223b-f7bd-4b26-ae2e-259db8d07fb6/d081cdcb-1181-4657-9580-dc3ba9a85775/ded358fb-ee52-4096-a32a-0cce52708100/0c7a1bf0-e6ae-42c1-a12c-9c71b98ed1be"
-					(reference "U903")
+					(reference "U901")
 					(unit 1)
 				)
@@
 		(dnp no)
 		(fields_autoplaced yes)
-		(property "Reference" "U901"
+		(property "Reference" "U903"
 			(at 63.1033 35.56 0)
 			(effects
@@
 			)
 		)
-		(property "Value" "74LS161"
+		(property "Value" "74HC161"
 			(at 63.1033 38.1 0)
 			(effects
@@
 			)
 		)
-		(property "Footprint" ""
+		(property "Footprint" "Package_DIP:DIP-16_W7.62mm"
 			(at 60.96 55.88 0)
 			(effects
@@
 			(project "BRISC8"
 				(path "/e198223b-f7bd-4b26-ae2e-259db8d07fb6/d081cdcb-1181-4657-9580-dc3ba9a85775/ded358fb-ee52-4096-a32a-0cce52708100/0c7a1bf0-e6ae-42c1-a12c-9c71b98ed1be"
-					(reference "U901")
+					(reference "U903")
 					(unit 1)
 				)
@@
 		(dnp no)
 		(fields_autoplaced yes)
-		(property "Reference" "U902"
+		(property "Reference" "U904"
 			(at 112.6333 35.56 0)
 			(effects
@@
 			)
 		)
-		(property "Value" "74LS161"
+		(property "Value" "74HC161"
 			(at 112.6333 38.1 0)
 			(effects
@@
 			)
 		)
-		(property "Footprint" ""
+		(property "Footprint" "Package_DIP:DIP-16_W7.62mm"
 			(at 110.49 55.88 0)
 			(effects
@@
 			(project "BRISC8"
 				(path "/e198223b-f7bd-4b26-ae2e-259db8d07fb6/d081cdcb-1181-4657-9580-dc3ba9a85775/ded358fb-ee52-4096-a32a-0cce52708100/0c7a1bf0-e6ae-42c1-a12c-9c71b98ed1be"
-					(reference "U902")
+					(reference "U904")
 					(unit 1)
 				)
@@
 			)
 		)
-		(property "Value" "C"
+		(property "Value" "0.1uF"
 			(at 151.13 184.1499 0)
 			(effects
@@
 			)
 		)
-		(property "Footprint" ""
+		(property "Footprint" "Capacitor_THT:C_Rect_L4.0mm_W2.5mm_P2.50mm"
 			(at 148.2852 186.69 0)
 			(effects
@@
 		(dnp no)
 		(fields_autoplaced yes)
-		(property "Reference" "#PWR0904"
+		(property "Reference" "#PWR0912"
 			(at 109.22 177.8 0)
 			(effects
@@
 			(project "BRISC8"
 				(path "/e198223b-f7bd-4b26-ae2e-259db8d07fb6/d081cdcb-1181-4657-9580-dc3ba9a85775/ded358fb-ee52-4096-a32a-0cce52708100/0c7a1bf0-e6ae-42c1-a12c-9c71b98ed1be"
-					(reference "#PWR0904")
+					(reference "#PWR0912")
 					(unit 1)
 				)
@@
 		(dnp no)
 		(fields_autoplaced yes)
-		(property "Reference" "#PWR0913"
+		(property "Reference" "#PWR0909"
 			(at 220.98 81.28 0)
 			(effects
@@
 			(project "BRISC8"
 				(path "/e198223b-f7bd-4b26-ae2e-259db8d07fb6/d081cdcb-1181-4657-9580-dc3ba9a85775/ded358fb-ee52-4096-a32a-0cce52708100/0c7a1bf0-e6ae-42c1-a12c-9c71b98ed1be"
-					(reference "#PWR0913")
+					(reference "#PWR0909")
 					(unit 1)
 				)
@@
 		(dnp no)
 		(fields_autoplaced yes)
-		(property "Reference" "#PWR0912"
+		(property "Reference" "#PWR0902"
 			(at 220.98 38.1 0)
 			(effects
@@
 			(project "BRISC8"
 				(path "/e198223b-f7bd-4b26-ae2e-259db8d07fb6/d081cdcb-1181-4657-9580-dc3ba9a85775/ded358fb-ee52-4096-a32a-0cce52708100/0c7a1bf0-e6ae-42c1-a12c-9c71b98ed1be"
-					(reference "#PWR0912")
+					(reference "#PWR0902")
 					(unit 1)
 				)
@@
 		(dnp no)
 		(fields_autoplaced yes)
-		(property "Reference" "U904"
+		(property "Reference" "U902"
 			(at 223.1233 34.29 0)
 			(effects
@@
 			)
 		)
-		(property "Footprint" ""
+		(property "Footprint" "Package_DIP:DIP-20_W7.62mm"
 			(at 220.98 54.61 0)
 			(effects
@@
 			(project "BRISC8"
 				(path "/e198223b-f7bd-4b26-ae2e-259db8d07fb6/d081cdcb-1181-4657-9580-dc3ba9a85775/ded358fb-ee52-4096-a32a-0cce52708100/0c7a1bf0-e6ae-42c1-a12c-9c71b98ed1be"
-					(reference "U904")
+					(reference "U902")
 					(unit 1)
 				)
@@
 			)
 		)
-		(property "Value" "C"
+		(property "Value" "0.1uF"
 			(at 138.43 184.1499 0)
 			(effects
@@
 			)
 		)
-		(property "Footprint" ""
+		(property "Footprint" "Capacitor_THT:C_Rect_L4.0mm_W2.5mm_P2.50mm"
 			(at 135.5852 186.69 0)
 			(effects
@@
 		(dnp no)
 		(fields_autoplaced yes)
-		(property "Reference" "#PWR0906"
+		(property "Reference" "#PWR0904"
 			(at 110.49 39.37 0)
 			(effects
@@
 			(project "BRISC8"
 				(path "/e198223b-f7bd-4b26-ae2e-259db8d07fb6/d081cdcb-1181-4657-9580-dc3ba9a85775/ded358fb-ee52-4096-a32a-0cce52708100/0c7a1bf0-e6ae-42c1-a12c-9c71b98ed1be"
-					(reference "#PWR0906")
+					(reference "#PWR0904")
 					(unit 1)
 				)
@@
 		(on_board yes)
 		(dnp no)
-		(property "Reference" "#PWR0908"
+		(property "Reference" "#PWR0906"
 			(at 148.59 68.58 0)
 			(effects
@@
 			(project "BRISC8"
 				(path "/e198223b-f7bd-4b26-ae2e-259db8d07fb6/d081cdcb-1181-4657-9580-dc3ba9a85775/ded358fb-ee52-4096-a32a-0cce52708100/0c7a1bf0-e6ae-42c1-a12c-9c71b98ed1be"
-					(reference "#PWR0908")
+					(reference "#PWR0906")
 					(unit 1)
 				)
@@
 		(dnp no)
 		(fields_autoplaced yes)
-		(property "Reference" "#PWR0905"
+		(property "Reference" "#PWR0913"
 			(at 109.22 198.12 0)
 			(effects
@@
 			(project "BRISC8"
 				(path "/e198223b-f7bd-4b26-ae2e-259db8d07fb6/d081cdcb-1181-4657-9580-dc3ba9a85775/ded358fb-ee52-4096-a32a-0cce52708100/0c7a1bf0-e6ae-42c1-a12c-9c71b98ed1be"
-					(reference "#PWR0905")
+					(reference "#PWR0913")
 					(unit 1)
 				)
